Commit message: 1day

File: urdf/arm_test.urdf (robot description, URDF)
Before this commit: robot test_robot, 5 links, 4 joints
Links:
- added link body3_link_yaw; visual box size=0.0 0.0 0.05
- added link world
- link base_link: geometry visual cylinder length=0.01 radius=0.02
- link body0_link_yaw: geometry visual box size=0.1 0.1 0.070
- link body1_link: geometry visual box size=0.1 0.1 0.480
- link body2_link: geometry visual box size=0.1 0.1 0.560
Joints:
- added joint body3_joint_yaw: type revolute, parent body2_link, child body3_link_yaw, origin xyz=0 0 0.560 rpy=0 0 0, axis 1 0 0, limit lower=-1.57075 upper=1.57075 effort=10000 velocity=1
- added joint fixed: type fixed, parent world, child base_link
- joint body0_joint_yaw: axis (none) -> 0 0 1; limit lower=-3.15 upper=3.15 effort=0 velocity=0 -> lower=-3.15 upper=3.15 effort=10000 velocity=1; origin xyz=0 0 0 rpy=0 1.5707 0 -> xyz=0 0 0 rpy=0 0 0
- joint body1_joint: axis (none) -> 0 1 0; limit lower=-10 upper=10 effort=0 velocity=0 -> lower=-1.57075 upper=1.57075 effort=10000 velocity=1; origin xyz=0 0 0 rpy=1.5707 -1.5707 -1.5707 -> xyz=0 0 0 rpy=0 0 0
- joint body2_joint: axis (none) -> 0 1 0; limit lower=-10 upper=10 effort=0 velocity=0 -> lower=-3.1415 upper=3.1415 effort=10000 velocity=1; origin xyz=0 0 0.5 rpy=0 0 0 -> xyz=0 0 0.480 rpy=0 0 0
- joint body3_joint: axis (none) -> 0 1 0; limit lower=-10 upper=10 effort=0 velocity=0 -> lower=-1.57075 upper=1.57075 effort=10000 velocity=1; origin xyz=0 0 0.4 rpy=0 0 0 -> xyz=0 0 0 rpy=0 0 0; parent body2_link -> body3_link_yaw
