Commit message: 0917

File: urdf/r5s_arm.urdf (robot description, URDF)
Before this commit: robot r5s, 9 links, 8 joints
Joints:
- joint body2_joint: limit lower=-3.15 upper=3.15 effort=0 velocity=100 -> lower=-0 upper=1.575 effort=0 velocity=100
- joint body3_joint: limit lower=-3.15 upper=3.15 effort=0 velocity=100 -> lower=-3.15 upper=0 effort=0 velocity=100
- joint body6_joint: limit lower=-3.15 upper=3.15 effort=0 velocity=100 -> lower=-31.5 upper=31.5 effort=0 velocity=100

Commit message: taikaino

File: urdf/r5s_arm.urdf (robot description, URDF)
Before this commit: robot r5s, 9 links, 8 joints
Joints:
- joint body6_joint: limit lower=-31.5 upper=31.5 effort=0 velocity=100 -> lower=-3.14159265 upper=3.14159265 effort=0 velocity=100

Commit message: Overlay

File: urdf/r5s_arm.urdf (robot description, URDF)
Before this commit: robot r5s, 9 links, 8 joints
Joints:
- joint body2_joint: limit lower=-0 upper=1.575 effort=0 velocity=100 -> lower=-0 upper=3.15 effort=0 velocity=100

Commit message: 1126

File: urdf/r5s_arm.urdf (robot description, URDF)
Before this commit: robot r5s, 9 links, 8 joints
Joints:
- joint body0_joint_yaw: limit lower=-3.15 upper=3.15 effort=0 velocity=100 -> lower=0 upper=0 effort=0 velocity=3.1415
- joint body1_joint: limit lower=-3.15 upper=3.15 effort=0 velocity=100 -> lower=-1.575 upper=1.575 effort=0 velocity=3.1415
- joint body2_joint: limit lower=-0 upper=3.15 effort=0 velocity=100 -> lower=-0 upper=3.15 effort=0 velocity=3.1415
- joint body3_joint: limit lower=-3.15 upper=0 effort=0 velocity=100 -> lower=-3.15 upper=0 effort=0 velocity=3.1415
- joint body4_joint: limit lower=-3.15 upper=3.15 effort=0 velocity=100 -> lower=-3.15 upper=3.15 effort=0 velocity=3.1415
- joint body5_joint: limit lower=-3.15 upper=3.15 effort=0 velocity=100 -> lower=-3.15 upper=3.15 effort=0 velocity=3.1415
- joint body6_joint: limit lower=-3.14159265 upper=3.14159265 effort=0 velocity=100 -> lower=-3.14159265 upper=3.14159265 effort=0 velocity=3.1415
